File: scr.brd (EAGLE design)
At the start: 99 x 70.8 mm, 58 parts, among them IC1 MEGA8-P, IC3 LM358N, Q1 16m, T2 BT148, T3 BT148

Commit message: upload
Parts:
- moved R14 56.1 mm to (69.8, 16.5), turned to 90 degrees
- moved T2 53.1 mm to (49.5, 22.9), turned to 0 degrees
- moved R5 52.5 mm to (43.2, 16.5), turned to 90 degrees
- moved OK1 48.7 mm to (61.0, 20.3), turned to 90 degrees
- moved R13 45.8 mm to (72.4, 16.5)
- moved T4 43.3 mm to (69.8, 6.35), turned to 270 degrees
- moved R4 36.8 mm to (54.6, 15.2), turned to 180 degrees
- moved T3 33.3 mm to (49.5, 12.7), turned to 0 degrees
- moved OK2 29.5 mm to (61.0, 10.2), turned to 90 degrees
- moved R9 16.5 mm to (54.6, 5.08), turned to 180 degrees
- moved T1 16.3 mm to (52.1, 26.7), turned to 0 degrees
- moved R8 5.68 mm to (68.6, 33.0), turned to 270 degrees
- moved R2 5.24 mm to (47.0, 30.5), turned to 0 degrees
- moved R18 3.81 mm to (39.4, 25.4)
Routing:
- net CTB: track 23.4 -> 77.3 mm, vias 0 -> 2
- net N$20: track 14.2 -> 67.2 mm
- net V-: track 10.7 -> 57.0 mm
- net CTA: track 27.6 -> 68.8 mm
- net V+: track 19.9 -> 57.8 mm
- net VCC: track 128.9 -> 146.0 mm
- net ZCDOUT: track 14.5 -> 0.00 mm
- net N$22: track 0.00 -> 6.88 mm
- net N$23: track 7.41 -> 2.54 mm
- net GND: track 562.0 -> 558.7 mm
- net N$7: track 3.81 -> 6.35 mm
- net TRIGER: track 41.7 -> 44.2 mm
- net N$3: track 2.54 -> 0.00 mm
- net ZCDIN: track 33.6 -> 32.1 mm
- net N$24: track 3.81 -> 5.08 mm
