File: scr.sch (EAGLE design)
At the start: 58 parts, among them IC1 MEGA8-P, IC3 LM358N, Q1 16m, T2 BT148, T3 BT148

Commit message: lagi
Parts:
- R11: value (none) -> 1k; device rcl:R-EU_0207/2V -> rcl:R-EU_0207/10
Connections:
- net N$11: now also R11.1; no longer R11.2
- net VREF: now also R11.2; no longer R11.1
Changed lines of the file:
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@@
 <part name="R26" library="rcl" deviceset="R-EU_" device="0207/2V"/>
 <part name="R12" library="rcl" deviceset="R-EU_" device="0207/2V"/>
-<part name="R11" library="rcl" deviceset="R-EU_" device="0207/2V"/>
 <part name="R8" library="rcl" deviceset="R-EU_" device="0207/10" value="10k"/>
 <part name="R10" library="rcl" deviceset="R-EU_" device="0207/2V"/>
 <part name="R2" library="rcl" deviceset="R-EU_" device="0207/2V"/>
 <part name="R18" library="rcl" deviceset="R-EU_" device="0207/2V"/>
+<part name="R11" library="rcl" deviceset="R-EU_" device="0207/10" value="1k"/>
 </parts>
 <sheets>
@@
 <instance part="R26" gate="G$1" x="111.76" y="-160.02"/>
 <instance part="R12" gate="G$1" x="121.92" y="-63.5"/>
-<instance part="R11" gate="G$1" x="91.44" y="-160.02"/>
 <instance part="R8" gate="G$1" x="96.52" y="-147.32" rot="MR180"/>
 <instance part="R10" gate="G$1" x="109.22" y="-119.38"/>
 <instance part="R2" gate="G$1" x="30.48" y="-10.16" rot="R90"/>
 <instance part="R18" gate="G$1" x="38.1" y="-5.08"/>
+<instance part="R11" gate="G$1" x="91.44" y="-160.02" rot="MR0"/>
 </instances>
 <busses>
@@
 <wire x1="109.22" y1="-152.4" x2="101.6" y2="-152.4" width="0.1524" layer="91"/>
 <pinref part="R26" gate="G$1" pin="1"/>
-<pinref part="R11" gate="G$1" pin="2"/>
+<pinref part="R11" gate="G$1" pin="1"/>
 </segment>
 </net>
@@
 <wire x1="86.36" y1="-160.02" x2="76.2" y2="-160.02" width="0.1524" layer="91"/>
 <label x="76.2" y="-160.02" size="1.778" layer="95" rot="R180" xref="yes"/>
-<pinref part="R11" gate="G$1" pin="1"/>
-</segment>
-</net>
+<pinref part="R11" gate="G$1" pin="2"/>
+</segment>
+</net>

Commit message: finish
Connections:
- removed net N$25: R16.1, X4-3.KL
- new net N$23: R16.1, X4-1.KL
- net GND: now also X4-3.KL; no longer X4-1.KL
Other:
- moved on the sheet: X4-1, X4-3
Changed lines of the file:
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@@
 <instance part="P+9" gate="VCC" x="160.02" y="93.98"/>
 <instance part="GND17" gate="1" x="160.02" y="73.66"/>
-<instance part="X4" gate="-1" x="165.1" y="-162.56" rot="R180"/>
+<instance part="X4" gate="-1" x="144.78" y="-109.22" rot="R180"/>
 <instance part="X4" gate="-2" x="162.56" y="-149.86" rot="R180"/>
-<instance part="X4" gate="-3" x="160.02" y="-109.22" rot="R180"/>
-<instance part="GND18" gate="1" x="157.48" y="-165.1"/>
+<instance part="X4" gate="-3" x="160.02" y="-160.02" rot="R180"/>
+<instance part="GND18" gate="1" x="154.94" y="-162.56"/>
 <instance part="R22" gate="G$1" x="220.98" y="63.5"/>
 <instance part="R23" gate="G$1" x="220.98" y="83.82"/>
@@
 </segment>
 <segment>
-<pinref part="X4" gate="-1" pin="KL"/>
-<pinref part="GND18" gate="1" pin="GND"/>
-<wire x1="157.48" y1="-162.56" x2="160.02" y2="-162.56" width="0.1524" layer="91"/>
-</segment>
-<segment>
 <pinref part="GND19" gate="1" pin="GND"/>
 <wire x1="213.36" y1="88.9" x2="213.36" y2="83.82" width="0.1524" layer="91"/>
@@
 <pinref part="R2" gate="G$1" pin="1"/>
 </segment>
+<segment>
+<pinref part="GND18" gate="1" pin="GND"/>
+<pinref part="X4" gate="-3" pin="KL"/>
+</segment>
 </net>
 <net name="N$3" class="0">
@@
 </segment>
 </net>
-<net name="N$25" class="0">
-<segment>
-<pinref part="R16" gate="G$1" pin="1"/>
-<wire x1="139.7" y1="-109.22" x2="154.94" y2="-109.22" width="0.1524" layer="91"/>
-<pinref part="X4" gate="-3" pin="KL"/>
-</segment>
-</net>
 <net name="N$26" class="0">
 <segment>
@@
 </segment>
 </net>
+<net name="N$23" class="0">
+<segment>
+<pinref part="R16" gate="G$1" pin="1"/>
+<pinref part="X4" gate="-1" pin="KL"/>
+</segment>
+</net>
