File: analog.brd (EAGLE design)
At the start: 160 x 100 mm, 23 parts, among them IC1 NE555, Q1 BC548A

Commit message: rout
Parts:
- moved C7 158.2 mm to (58.4, 35.6)
- moved C8 142.0 mm to (39.4, 24.1)
- moved R8 124.8 mm to (71.1, 22.9)
- moved C6 119.5 mm to (35.6, 11.4)
- moved D3 107.2 mm to (47.0, 11.4)
- moved IC2 106.1 mm to (25.4, 14.0)
- moved D2 105.2 mm to (47.0, 14.0)
- moved C5 101.0 mm to (30.5, 5.08), turned to 270 degrees
- moved R7 90.4 mm to (43.2, 33.0), turned to 180 degrees
- moved D1 79.5 mm to (17.8, 33.0)
- moved R4 78.8 mm to (43.2, 27.9)
- moved C3 72.3 mm to (30.5, 19.1), turned to 180 degrees
- moved Q1 70.9 mm to (8.89, 35.6), turned to 270 degrees
- moved C2 69.9 mm to (39.4, 19.1), turned to 180 degrees
- moved R5 63.7 mm to (43.2, 30.5)
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Routing:
- net VCC: track 0.00 -> 28.8 mm
- net N$5: track 0.00 -> 6.35 mm

Commit message: finish sch
Parts:
- removed R3: 39k, rcl:0207/10
- added C1: 100nF, rcl:C050-025X075
- added LSP1, LSP2, LSP3, LSP4, LSP5: MCS10B, solpad:MCS10B
- added R10, R9: 10, rcl:0207/10
- added R11: 1k, rcl:0207/10
- added R12, R13: 39k, rcl:0207/10
- added T1, T2: BTV58, triac:TO220CS
- added X1, X3, X4, X7: (no value), con-wago-500:W237-103
- added X2, X5, X6: (no value), con-wago-500:W237-102
- C4: value 2.2uF -> 100nF; device rcl:E5-8,5 -> rcl:C050-025X075
- C5: value 2.2uF -> 1000uF/25v
- C8: value (none) -> 2,2uF/16v
- moved C4 156.4 mm to (85.1, 53.3), turned to 90 degrees
- moved D4 118.7 mm to (7.62, 55.9), turned to 90 degrees
Connections:
- new net N$11: R1.2, X2.1
- new net N$14: OK1.2, X2.2
- new net N$15: LSP2.MP, R8.2
- new net N$16: R12.2, X4.1
- new net N$17: LSP3.MP, X5.2
- new net N$18: LSP5.MP, X5.1
- new net N$19: C1.1, R9.1
- new net N$20: C1.2, T1.A, X7.3
- new net N$21: R10.2, R11.1, R9.2, T1.C, T2.C, X4.2, X6.2, X7.2
- new net N$22: C4.1, R10.1
- new net N$23: C4.2, T2.A, X7.1
- new net N$24: R13.2, X4.3
- new net N$25: R12.1, T1.G
- new net N$26: R13.1, T2.G
- net GND: now also R11.2, X3.2, X6.1; no longer OK1.2
- net N$10: no longer R1.2
- net N$12: now also X3.1
- net N$13: now also X3.3
- net N$5: now also X1.2, X1.3
- net N$9: now also LSP1.MP
- net VCC: now also OK1.5, X1.1

Commit message: routing
Parts:
- moved R12 69.0 mm to (47.0, 30.5), turned to 0 degrees
- moved R13 67.3 mm to (53.3, 33.0), turned to 180 degrees
- moved X7 64.9 mm to (59.7, 39.4), turned to 180 degrees
- moved X4 61.1 mm to (44.5, 39.4), turned to 180 degrees
- moved LSP2 55.3 mm to (61.0, 3.81), turned to 270 degrees
- moved LSP5 52.8 mm to (71.1, 3.81)
- moved LSP4 51.1 mm to (71.1, 8.89)
- moved LSP3 50.3 mm to (71.1, 14.0)
- moved LSP1 50.3 mm to (61.0, 14.0), turned to 270 degrees
- moved Q1 48.2 mm to (54.6, 20.3), turned to 0 degrees
- moved D1 41.9 mm to (52.1, 8.89), turned to 90 degrees
- moved X5 41.0 mm to (81.3, 7.62)
- moved D2 37.1 mm to (24.1, 43.2), turned to 180 degrees
- moved D3 37.1 mm to (24.1, 40.6), turned to 180 degrees
- moved T1 34.1 mm to (64.8, 24.1), turned to 180 degrees
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Connections:
- new net N$27: R10.2, R11.1, R9.2, T1.C, T2.C, X4.2, X6.2
- net GND: no longer R11.2, X6.1
- net N$21: now also R11.2, X6.1; no longer R10.2, R11.1, R9.2, T1.C, T2.C, X4.2, X6.2
Routing:
- net GND: track 0.00 -> 333.6 mm
- net N$27: track 0.00 -> 96.8 mm
- net N$21: track 0.00 -> 63.1 mm
- net VCC: track 28.8 -> 65.2 mm
- net N$5: track 6.35 -> 34.6 mm
- net N$20: track 0.00 -> 27.7 mm
- net N$25: track 0.00 -> 21.9 mm
- net N$9: track 0.00 -> 21.2 mm
- net N$2: track 0.00 -> 20.6 mm
- net N$14: track 0.00 -> 16.6 mm
- net N$24: track 0.00 -> 15.9 mm
- net N$6: track 0.00 -> 15.5 mm
- net +12V: track 0.00 -> 15.0 mm
- net N$22: track 0.00 -> 15.0 mm
- net N$13: track 0.00 -> 13.8 mm
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- added copper zone on layer 16, net GND
Other:
- board size 160 x 100 mm -> 85.1 x 47.9 mm
