File: analog.sch (EAGLE design)
At the start: 23 parts, among them IC1 NE555, Q1 BC548A

Commit message: finish sch
Parts:
- removed R3: 39k, rcl:R-EU_0207/10
- added C1: 100nF, rcl:C-EU050-025X075
- added LSP1, LSP2, LSP3, LSP4, LSP5: MCS10B, solpad:MCS10B
- added R10, R9: 10, rcl:R-EU_0207/10
- added R11: 1k, rcl:R-EU_0207/10
- added R12, R13: 39k, rcl:R-EU_0207/10
- added T1, T2: BTV58, triac:BTV58
- added X1, X3, X4, X7: (no value), con-wago-500:W237-103
- added X2, X5, X6: (no value), con-wago-500:W237-102
- C4: value 2.2uF -> 100nF; device rcl:CPOL-EUE5-8.5 -> rcl:C-EU050-025X075
- C5: value 2.2uF -> 1000uF/25v
- C8: value (none) -> 2,2uF/16v
Connections:
- new net N$11: R1.2, X2-1.KL
- new net N$14: OK1.C, X2-2.KL
- new net N$15: LSP2.MP, R8.2
- new net N$16: R12.2, X4-1.KL
- new net N$17: LSP3.MP, X5-2.KL
- new net N$18: LSP5.MP, X5-1.KL
- new net N$19: C1.1, R9.1
- new net N$20: C1.2, T1.A, X7-3.KL
- new net N$21: R10.2, R11.1, R9.2, T1.C, T2.C, X4-2.KL, X6-2.KL, X7-2.KL
- new net N$22: C4.1, R10.1
- new net N$23: C4.2, T2.A, X7-1.KL
- new net N$24: R13.2, X4-3.KL
- new net N$25: R12.1, T1.G
- new net N$26: R13.1, T2.G
- net GND: now also R11.2, X3-2.KL, X6-1.KL; no longer OK1.C
- net N$10: no longer R1.2
- net N$12: now also X3-1.KL
- net N$13: now also X3-3.KL
- net N$5: now also X1-2.KL, X1-3.KL
- net N$9: now also LSP1.MP
- net VCC: now also OK1.COL, X1-1.KL
Other:
- moved on the sheet: D2, D3, R1

Commit message: routing
Connections:
- new net N$27: R10.2, R11.1, R9.2, T1.C, T2.C, X4-2.KL, X6-2.KL
- net GND: no longer R11.2, X6-1.KL
- net N$21: now also R11.2, X6-1.KL; no longer R10.2, R11.1, R9.2, T1.C, T2.C, X4-2.KL, X6-2.KL
Changed lines of the file:
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@@
 <part name="R10" library="rcl" deviceset="R-EU_" device="0207/10" value="10"/>
 <part name="R11" library="rcl" deviceset="R-EU_" device="0207/10" value="1k"/>
-<part name="GND11" library="supply1" deviceset="GND" device=""/>
 <part name="X4" library="con-wago-500" deviceset="W237-103" device=""/>
 <part name="X5" library="con-wago-500" deviceset="W237-102" device=""/>
@@
 <instance part="R10" gate="G$1" x="73.66" y="2.54" rot="R270"/>
 <instance part="R11" gate="G$1" x="73.66" y="-22.86" rot="R270"/>
-<instance part="GND11" gate="1" x="73.66" y="-38.1"/>
 <instance part="X4" gate="-1" x="20.32" y="-20.32"/>
 <instance part="X4" gate="-2" x="20.32" y="-25.4"/>
@@
 <wire x1="-193.04" y1="17.78" x2="-195.58" y2="17.78" width="0.1524" layer="91"/>
 </segment>
-<segment>
-<pinref part="R11" gate="G$1" pin="2"/>
-<pinref part="GND11" gate="1" pin="GND"/>
-<wire x1="73.66" y1="-35.56" x2="73.66" y2="-30.48" width="0.1524" layer="91"/>
-<pinref part="X6" gate="-1" pin="KL"/>
-<wire x1="73.66" y1="-30.48" x2="73.66" y2="-27.94" width="0.1524" layer="91"/>
-<junction x="73.66" y="-30.48"/>
-</segment>
 </net>
 <net name="N$5" class="0">
@@
 </segment>
 </net>
-<net name="N$21" class="0">
+<net name="N$22" class="0">
+<segment>
+<pinref part="C4" gate="G$1" pin="1"/>
+<pinref part="R10" gate="G$1" pin="1"/>
+</segment>
+</net>
+<net name="N$23" class="0">
+<segment>
+<pinref part="T2" gate="1" pin="A"/>
+<wire x1="58.42" y1="7.62" x2="58.42" y2="20.32" width="0.1524" layer="91"/>
+<pinref part="C4" gate="G$1" pin="2"/>
+<wire x1="58.42" y1="20.32" x2="66.04" y2="20.32" width="0.1524" layer="91"/>
+<wire x1="66.04" y1="20.32" x2="73.66" y2="20.32" width="0.1524" layer="91"/>
+<wire x1="73.66" y1="20.32" x2="73.66" y2="15.24" width="0.1524" layer="91"/>
+<junction x="66.04" y="20.32"/>
+<pinref part="X7" gate="-1" pin="KL"/>
+<wire x1="22.86" y1="43.18" x2="66.04" y2="43.18" width="0.1524" layer="91"/>
+<wire x1="66.04" y1="43.18" x2="66.04" y2="20.32" width="0.1524" layer="91"/>
+</segment>
+</net>
+<net name="N$25" class="0">
+<segment>
+<pinref part="T1" gate="1" pin="G"/>
+<pinref part="R12" gate="G$1" pin="1"/>
+<wire x1="25.4" y1="2.54" x2="27.94" y2="2.54" width="0.1524" layer="91"/>
+</segment>
+</net>
+<net name="N$16" class="0">
+<segment>
+<pinref part="R12" gate="G$1" pin="2"/>
+<pinref part="X4" gate="-1" pin="KL"/>
+<wire x1="25.4" y1="-20.32" x2="25.4" y2="-7.62" width="0.1524" layer="91"/>
+</segment>
+</net>
+<net name="N$24" class="0">
+<segment>
+<pinref part="R13" gate="G$1" pin="2"/>
+<pinref part="X4" gate="-3" pin="KL"/>
+<wire x1="25.4" y1="-30.48" x2="55.88" y2="-30.48" width="0.1524" layer="91"/>
+<wire x1="55.88" y1="-30.48" x2="55.88" y2="-22.86" width="0.1524" layer="91"/>
+</segment>
+</net>
+<net name="N$26" class="0">
+<segment>
+<pinref part="T2" gate="1" pin="G"/>
+<pinref part="R13" gate="G$1" pin="1"/>
+<wire x1="55.88" y1="2.54" x2="55.88" y2="-12.7" width="0.1524" layer="91"/>
+</segment>
+</net>
+<net name="N$27" class="0">
 <segment>
 <pinref part="T1" gate="1" pin="C"/>
@@
 <wire x1="58.42" y1="-7.62" x2="73.66" y2="-7.62" width="0.1524" layer="91"/>
 <wire x1="73.66" y1="-7.62" x2="73.66" y2="-2.54" width="0.1524" layer="91"/>
-<wire x1="45.72" y1="-7.62" x2="50.8" y2="-7.62" width="0.1524" layer="91"/>
 <pinref part="R11" gate="G$1" pin="1"/>
-<wire x1="50.8" y1="-7.62" x2="58.42" y2="-7.62" width="0.1524" layer="91"/>
+<wire x1="45.72" y1="-7.62" x2="58.42" y2="-7.62" width="0.1524" layer="91"/>
 <wire x1="73.66" y1="-7.62" x2="73.66" y2="-12.7" width="0.1524" layer="91"/>
 <pinref part="X4" gate="-2" pin="KL"/>
@@
 <pinref part="X6" gate="-2" pin="KL"/>
 <junction x="73.66" y="-12.7"/>
+<junction x="45.72" y="-7.62"/>
+<junction x="58.42" y="-7.62"/>
+</segment>
+</net>
+<net name="N$21" class="0">
+<segment>
 <pinref part="X7" gate="-2" pin="KL"/>
 <wire x1="22.86" y1="35.56" x2="50.8" y2="35.56" width="0.1524" layer="91"/>
-<wire x1="50.8" y1="35.56" x2="50.8" y2="-7.62" width="0.1524" layer="91"/>
-<junction x="45.72" y="-7.62"/>
-<junction x="50.8" y="-7.62"/>
-<junction x="58.42" y="-7.62"/>
-</segment>
-</net>
-<net name="N$22" class="0">
-<segment>
-<pinref part="C4" gate="G$1" pin="1"/>
-<pinref part="R10" gate="G$1" pin="1"/>
-</segment>
-</net>
-<net name="N$23" class="0">
-<segment>
-<pinref part="T2" gate="1" pin="A"/>
-<wire x1="58.42" y1="7.62" x2="58.42" y2="20.32" width="0.1524" layer="91"/>
-<pinref part="C4" gate="G$1" pin="2"/>
-<wire x1="58.42" y1="20.32" x2="66.04" y2="20.32" width="0.1524" layer="91"/>
-<wire x1="66.04" y1="20.32" x2="73.66" y2="20.32" width="0.1524" layer="91"/>
-<wire x1="73.66" y1="20.32" x2="73.66" y2="15.24" width="0.1524" layer="91"/>
-<junction x="66.04" y="20.32"/>
-<pinref part="X7" gate="-1" pin="KL"/>
-<wire x1="22.86" y1="43.18" x2="66.04" y2="43.18" width="0.1524" layer="91"/>
-<wire x1="66.04" y1="43.18" x2="66.04" y2="20.32" width="0.1524" layer="91"/>
-</segment>
-</net>
-<net name="N$25" class="0">
-<segment>
-<pinref part="T1" gate="1" pin="G"/>
-<pinref part="R12" gate="G$1" pin="1"/>
-<wire x1="25.4" y1="2.54" x2="27.94" y2="2.54" width="0.1524" layer="91"/>
-</segment>
-</net>
-<net name="N$16" class="0">
-<segment>
-<pinref part="R12" gate="G$1" pin="2"/>
-<pinref part="X4" gate="-1" pin="KL"/>
-<wire x1="25.4" y1="-20.32" x2="25.4" y2="-7.62" width="0.1524" layer="91"/>
-</segment>
-</net>
-<net name="N$24" class="0">
-<segment>
-<pinref part="R13" gate="G$1" pin="2"/>
-<pinref part="X4" gate="-3" pin="KL"/>
-<wire x1="25.4" y1="-30.48" x2="55.88" y2="-30.48" width="0.1524" layer="91"/>
-<wire x1="55.88" y1="-30.48" x2="55.88" y2="-22.86" width="0.1524" layer="91"/>
-</segment>
-</net>
-<net name="N$26" class="0">
-<segment>
-<pinref part="T2" gate="1" pin="G"/>
-<pinref part="R13" gate="G$1" pin="1"/>
-<wire x1="55.88" y1="2.54" x2="55.88" y2="-12.7" width="0.1524" layer="91"/>
-</segment>
-</net>
+<wire x1="50.8" y1="35.56" x2="50.8" y2="-35.56" width="0.1524" layer="91"/>
+<pinref part="R11" gate="G$1" pin="2"/>
+<pinref part="X6" gate="-1" pin="KL"/>
+<wire x1="73.66" y1="-30.48" x2="73.66" y2="-27.94" width="0.1524" layer="91"/>
+<wire x1="50.8" y1="-35.56" x2="73.66" y2="-35.56" width="0.1524" layer="91"/>
+<wire x1="73.66" y1="-35.56" x2="73.66" y2="-30.48" width="0.1524" layer="91"/>
+<junction x="73.66" y="-30.48"/>
+</segment>
+</net>
