File: controler scr.brd (EAGLE design)
At the start: 71.1 x 56.8 mm, 31 parts, among them IC1 MEGA8-P, Q1 16m, Q2 TIP41C, T2 BT148

Commit message: revisi
Parts:
- added D5: 1N4002, diode:DO35-10
Connections:
- removed net AVCC: IC1.20
- new net N$3: D5.C, T2.G
- net N$9: now also D5.A; no longer T2.G
- net VCC: now also IC1.20
Routing:
- net N$9: track 46.9 -> 76.5 mm, vias 0 -> 2
- net VCC: track 63.8 -> 73.3 mm
- net GND: track 415.0 -> 406.3 mm
- net N$3: track 0.00 -> 5.71 mm
Changed lines of the file:
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@@
 <element name="R7" library="rcl" package="0207/10" value="100" x="29.21" y="39.37" rot="R180"/>
 <element name="R6" library="rcl" package="0207/10" value="100" x="13.97" y="25.4" rot="R180"/>
+<element name="D5" library="diode" package="DO35-10" value="1N4002" x="54.61" y="21.59"/>
 </elements>
 <signals>
@@
 <wire x1="41.91" y1="26.67" x2="40.64" y2="27.94" width="0.8128" layer="16"/>
 <wire x1="40.64" y1="27.94" x2="40.64" y2="30.48" width="0.8128" layer="16"/>
-<wire x1="45.72" y1="52.07" x2="45.72" y2="49.53" width="0.8128" layer="16"/>
-<wire x1="45.72" y1="49.53" x2="48.26" y2="46.99" width="0.8128" layer="16"/>
-<wire x1="48.26" y1="44.45" x2="48.26" y2="46.99" width="0.8128" layer="16"/>
 <wire x1="59.69" y1="13.97" x2="69.85" y2="13.97" width="0.8128" layer="16"/>
 <contactref element="X2" pad="6"/>
@@
 <wire x1="24.13" y1="36.83" x2="24.13" y2="39.37" width="0.8128" layer="16"/>
 <wire x1="24.13" y1="39.37" x2="24.13" y2="45.72" width="0.8128" layer="16"/>
+<contactref element="IC1" pad="20"/>
+<wire x1="50.8" y1="52.07" x2="50.8" y2="48.26" width="0.6096" layer="16"/>
+<wire x1="50.8" y1="48.26" x2="49.53" y2="46.99" width="0.6096" layer="16"/>
+<wire x1="49.53" y1="46.99" x2="45.72" y2="46.99" width="0.6096" layer="16"/>
 </signal>
 <signal name="N$1">
@@
 <signal name="N$9">
 <contactref element="OK1" pad="3"/>
-<contactref element="T2" pad="G"/>
 <contactref element="X2" pad="2"/>
-<wire x1="45.72" y1="23.876" x2="30.226" y2="23.876" width="0.8128" layer="16"/>
-<wire x1="30.226" y1="23.876" x2="29.21" y2="22.86" width="0.8128" layer="16"/>
-<wire x1="29.21" y1="22.86" x2="29.21" y2="13.97" width="0.8128" layer="16"/>
 <wire x1="29.21" y1="13.97" x2="35.56" y2="7.62" width="0.8128" layer="16"/>
 <wire x1="35.56" y1="7.62" x2="35.56" y2="6.47" width="0.8128" layer="16"/>
 <wire x1="35.56" y1="6.47" x2="35.68" y2="6.35" width="0.8128" layer="16"/>
-<wire x1="45.72" y1="23.876" x2="53.086" y2="23.876" width="0.8128" layer="16"/>
-<wire x1="53.086" y1="23.876" x2="54.61" y2="25.4" width="0.8128" layer="16"/>
-<wire x1="54.61" y1="25.4" x2="54.61" y2="26.67" width="0.8128" layer="16"/>
+<contactref element="D5" pad="A"/>
+<wire x1="59.69" y1="21.59" x2="62.23" y2="24.13" width="0.6096" layer="16"/>
+<wire x1="62.23" y1="24.13" x2="62.23" y2="27.94" width="0.6096" layer="16"/>
+<wire x1="62.23" y1="27.94" x2="59.69" y2="30.48" width="0.6096" layer="16"/>
+<wire x1="54.61" y1="26.67" x2="53.34" y2="26.67" width="0.6096" layer="16"/>
+<wire x1="53.34" y1="26.67" x2="52.07" y2="27.94" width="0.6096" layer="16"/>
+<wire x1="52.07" y1="27.94" x2="52.07" y2="29.21" width="0.6096" layer="16"/>
+<wire x1="52.07" y1="29.21" x2="53.34" y2="30.48" width="0.6096" layer="16"/>
+<wire x1="53.34" y1="30.48" x2="59.69" y2="30.48" width="0.6096" layer="16"/>
+<via x="29.21" y="13.97" extent="1-16" drill="0.6" diameter="1.6764" shape="octagon"/>
+<wire x1="29.21" y1="13.97" x2="34.29" y2="13.97" width="0.6096" layer="1"/>
+<wire x1="34.29" y1="13.97" x2="38.1" y2="10.16" width="0.6096" layer="1"/>
+<wire x1="38.1" y1="10.16" x2="53.34" y2="10.16" width="0.6096" layer="1"/>
+<wire x1="53.34" y1="10.16" x2="54.61" y2="11.43" width="0.6096" layer="1"/>
+<wire x1="54.61" y1="11.43" x2="54.61" y2="24.13" width="0.6096" layer="1"/>
+<via x="54.61" y="24.13" extent="1-16" drill="0.6" diameter="1.6764" shape="octagon"/>
+<wire x1="54.61" y1="24.13" x2="54.61" y2="26.67" width="0.6096" layer="16"/>
 </signal>
 <signal name="N$10">
@@
 <wire x1="50.8" y1="6.47" x2="50.68" y2="6.35" width="0.8128" layer="16"/>
 </signal>
-<signal name="AVCC">
-<contactref element="IC1" pad="20"/>
-</signal>
 <signal name="N$7">
 <contactref element="OK3" pad="4"/>
@@
 <wire x1="22.86" y1="17.78" x2="22.86" y2="22.86" width="0.8128" layer="16"/>
 </signal>
+<signal name="N$3">
+<contactref element="T2" pad="G"/>
+<contactref element="D5" pad="C"/>
+<wire x1="49.53" y1="21.59" x2="49.53" y2="22.86" width="0.6096" layer="16"/>
+<wire x1="49.53" y1="22.86" x2="48.26" y2="24.13" width="0.6096" layer="16"/>
+<wire x1="48.26" y1="24.13" x2="45.974" y2="24.13" width="0.6096" layer="16"/>
+<wire x1="45.974" y1="24.13" x2="45.72" y2="23.876" width="0.6096" layer="16"/>
+</signal>
 </signals>
