File: controler scr.sch (EAGLE design)
At the start: 31 parts, among them IC1 MEGA8-P, Q1 16m, Q2 TIP41C, T2 BT148

Commit message: revisi
Parts:
- added D5: 1N4002, diode:1N4446
Connections:
- new net N$3: D5.C, T2.G
- net N$9: now also D5.A; no longer T2.G
- net VCC: now also IC1.AVCC
Changed lines of the file:
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@@
 <part name="P+7" library="supply1" deviceset="+12V" device=""/>
 <part name="GND15" library="supply1" deviceset="GND" device=""/>
+<part name="D5" library="diode" deviceset="1N4446" device="" value="1N4002"/>
 </parts>
 <sheets>
@@
 <instance part="P+7" gate="1" x="167.64" y="-20.32"/>
 <instance part="GND15" gate="1" x="236.22" y="22.86" rot="R270"/>
+<instance part="D5" gate="1" x="170.18" y="-43.18" smashed="yes">
+<attribute name="NAME" x="162.56" y="-40.1574" size="1.778" layer="95"/>
+<attribute name="VALUE" x="167.64" y="-40.4114" size="1.778" layer="96"/>
+</instance>
 </instances>
 <busses>
@@
 <wire x1="73.66" y1="86.36" x2="73.66" y2="71.12" width="0.1524" layer="91"/>
 <pinref part="P+4" gate="VCC" pin="VCC"/>
+<pinref part="IC1" gate="G$1" pin="AVCC"/>
+<wire x1="91.44" y1="60.96" x2="73.66" y2="60.96" width="0.1524" layer="91"/>
+<wire x1="73.66" y1="60.96" x2="73.66" y2="71.12" width="0.1524" layer="91"/>
+<junction x="73.66" y="71.12"/>
 </segment>
 <segment>
@@
 <segment>
 <pinref part="OK1" gate="A" pin="EMIT"/>
-<pinref part="T2" gate="1" pin="G"/>
 <wire x1="162.56" y1="-43.18" x2="167.64" y2="-43.18" width="0.1524" layer="91"/>
 <pinref part="X2" gate="-2" pin="KL"/>
-<wire x1="167.64" y1="-43.18" x2="172.72" y2="-43.18" width="0.1524" layer="91"/>
 <wire x1="167.64" y1="-53.34" x2="167.64" y2="-43.18" width="0.1524" layer="91"/>
+<pinref part="D5" gate="1" pin="A"/>
 <junction x="167.64" y="-43.18"/>
 </segment>
@@
 </segment>
 </net>
+<net name="N$3" class="0">
+<segment>
+<pinref part="T2" gate="1" pin="G"/>
+<pinref part="D5" gate="1" pin="C"/>
+</segment>
+</net>
