File: display.brd (EAGLE design)
At the start: 82.5 x 64.8 mm, 36 parts, among them IC1 MEGA8-P

Commit message: revisi
Parts:
- moved SV1 3.59 mm to (12.7, 5.08)
Routing:
- net N$21: track 8.67 -> 12.3 mm
- net N$13: track 8.67 -> 12.3 mm
- net N$11: track 8.67 -> 12.3 mm
- net GND: track 381.3 -> 378.8 mm
Changed lines of the file:
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@@
 <dimension x1="-2.54" y1="67.31" x2="-2.54" y2="1.27" x3="-8.89" y3="34.29" textsize="1.778" layer="21"/>
 <dimension x1="-2.54" y1="67.31" x2="80.01" y2="67.31" x3="38.735" y3="69.85" textsize="1.778" layer="21"/>
-<dimension x1="62.23" y1="50.8" x2="62.23" y2="60.96" x3="87.63" y3="55.88" textsize="1.778" layer="21"/>
-<dimension x1="62.23" y1="50.8" x2="62.23" y2="6.35" x3="90.17" y3="28.575" textsize="1.778" layer="21"/>
-<dimension x1="74.93" y1="60.96" x2="43.18" y2="60.96" x3="59.055" y3="76.2" textsize="1.778" layer="21"/>
-<dimension x1="2.54" y1="60.96" x2="43.18" y2="60.96" x3="22.86" y3="76.2" textsize="1.778" layer="21"/>
 </plain>
 <attributes>
@@
 </element>
 <element name="R1" library="rcl" package="0207/7" value="330" x="10.16" y="12.7"/>
-<element name="SV1" library="con-lstb" package="MA04-1" value="" x="10.16" y="7.62">
-<attribute name="OC_NEWARK" value="unknown" x="10.16" y="7.62" size="1.778" layer="27" display="off"/>
-<attribute name="MF" value="" x="10.16" y="7.62" size="1.778" layer="27" display="off"/>
-<attribute name="MPN" value="" x="10.16" y="7.62" size="1.778" layer="27" display="off"/>
-<attribute name="OC_FARNELL" value="unknown" x="10.16" y="7.62" size="1.778" layer="27" display="off"/>
+<element name="SV1" library="con-lstb" package="MA04-1" value="" x="12.7" y="5.08">
+<attribute name="OC_NEWARK" value="unknown" x="12.7" y="5.08" size="1.778" layer="27" display="off"/>
+<attribute name="MF" value="" x="12.7" y="5.08" size="1.778" layer="27" display="off"/>
+<attribute name="MPN" value="" x="12.7" y="5.08" size="1.778" layer="27" display="off"/>
+<attribute name="OC_FARNELL" value="unknown" x="12.7" y="5.08" size="1.778" layer="27" display="off"/>
 </element>
 <element name="SV2" library="con-lstb" package="MA04-1" value="" x="49.53" y="7.62">
@@
 <wire x1="11.43" y1="64.77" x2="-1.27" y2="64.77" width="0.6096" layer="16"/>
 <wire x1="-1.27" y1="64.77" x2="-1.27" y2="2.54" width="0.6096" layer="16"/>
-<wire x1="-1.27" y1="2.54" x2="6.35" y2="2.54" width="0.6096" layer="16"/>
-<wire x1="6.35" y1="2.54" x2="26.67" y2="2.54" width="0.6096" layer="16"/>
+<wire x1="-1.27" y1="2.54" x2="8.89" y2="2.54" width="0.6096" layer="16"/>
+<wire x1="8.89" y1="2.54" x2="26.67" y2="2.54" width="0.6096" layer="16"/>
 <wire x1="66.04" y1="20.32" x2="78.74" y2="20.32" width="0.6096" layer="16"/>
 <contactref element="SV1" pad="1"/>
@@
 </polygon>
 <wire x1="78.74" y1="52.07" x2="64.77" y2="52.07" width="0.6096" layer="16"/>
-<wire x1="6.35" y1="7.62" x2="6.35" y2="2.54" width="0.6096" layer="16"/>
+<wire x1="8.89" y1="5.08" x2="8.89" y2="2.54" width="0.6096" layer="16"/>
 </signal>
 <signal name="VCC">
@@
 <contactref element="SV1" pad="2"/>
 <wire x1="6.35" y1="12.7" x2="6.35" y2="11.43" width="0.6096" layer="16"/>
-<wire x1="6.35" y1="11.43" x2="7.62" y2="10.16" width="0.6096" layer="16"/>
-<wire x1="7.62" y1="10.16" x2="8.89" y2="8.89" width="0.6096" layer="16"/>
-<wire x1="8.89" y1="8.89" x2="8.89" y2="7.62" width="0.6096" layer="16"/>
+<wire x1="6.35" y1="11.43" x2="11.43" y2="6.35" width="0.6096" layer="16"/>
+<wire x1="11.43" y1="6.35" x2="11.43" y2="5.08" width="0.6096" layer="16"/>
 </signal>
 <signal name="N$11">
 <contactref element="SV1" pad="3"/>
 <contactref element="IC1" pad="2"/>
-<wire x1="11.43" y1="7.62" x2="11.43" y2="8.89" width="0.6096" layer="16"/>
-<wire x1="11.43" y1="8.89" x2="8.89" y2="11.43" width="0.6096" layer="16"/>
+<wire x1="13.97" y1="5.08" x2="13.97" y2="6.35" width="0.6096" layer="16"/>
+<wire x1="13.97" y1="6.35" x2="8.89" y2="11.43" width="0.6096" layer="16"/>
 <wire x1="8.89" y1="11.43" x2="8.89" y2="15.24" width="0.6096" layer="16"/>
 </signal>
@@
 <contactref element="IC1" pad="3"/>
 <contactref element="SV1" pad="4"/>
-<wire x1="13.97" y1="7.62" x2="13.97" y2="8.89" width="0.6096" layer="16"/>
-<wire x1="13.97" y1="8.89" x2="11.43" y2="11.43" width="0.6096" layer="16"/>
+<wire x1="16.51" y1="5.08" x2="16.51" y2="6.35" width="0.6096" layer="16"/>
+<wire x1="16.51" y1="6.35" x2="11.43" y2="11.43" width="0.6096" layer="16"/>
 <wire x1="11.43" y1="11.43" x2="11.43" y2="15.24" width="0.6096" layer="16"/>
 </signal>
