File: display.sch (EAGLE design)
At the start: 36 parts, among them IC1 MEGA8-P

Commit message: reset display
Parts:
- removed H1, H2, H3, H4: MOUNT-PAD-ROUND3.0, holes:MOUNT-PAD-ROUND3.0
Changed lines of the file:
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@@
 <part name="R11" library="rcl" deviceset="R-EU_" device="0207/7" value="330"/>
 <part name="GND3" library="supply1" deviceset="GND" device=""/>
-<part name="H1" library="holes" deviceset="MOUNT-PAD-ROUND" device="3.0"/>
-<part name="H2" library="holes" deviceset="MOUNT-PAD-ROUND" device="3.0"/>
-<part name="H3" library="holes" deviceset="MOUNT-PAD-ROUND" device="3.0"/>
-<part name="H4" library="holes" deviceset="MOUNT-PAD-ROUND" device="3.0"/>
 </parts>
 <sheets>
@@
 <instance part="R11" gate="G$1" x="147.32" y="76.2" rot="R270"/>
 <instance part="GND3" gate="1" x="139.7" y="68.58"/>
-<instance part="H1" gate="G$1" x="20.32" y="55.88"/>
-<instance part="H2" gate="G$1" x="20.32" y="50.8"/>
-<instance part="H3" gate="G$1" x="20.32" y="45.72"/>
-<instance part="H4" gate="G$1" x="20.32" y="40.64"/>
 </instances>
 <busses>
